Commit message: Imported upstream version '0.2.2' of 'upstream'

File: mrp2_description/urdf/base/base.urdf.xacro (robot description, xacro)
@@ -7,6 +7,7 @@
   <xacro:include filename="$(find mrp2_description)/urdf/sensors/hokuyo_utm_30lx_laser.urdf.xacro"/>
   <xacro:include filename="$(find mrp2_description)/urdf/sensors/imu.urdf.xacro"/>
+  <xacro:include filename="$(find mrp2_description)/urdf/sensors/sonar.urdf.xacro"/>
   <!-- Wheel characteristics -->
-  <property name="wheel_radius"     value="0.102"/>
+  <property name="wheel_radius"     value="0.100"/>
   <property name="wheel_width"      value="0.050"/>
   <property name="wheel_separation" value="0.478"/>
@@ -70,5 +71,5 @@
     </xacro:hokuyo_utm_30lx_laser>
     <!-- IMU -->
-    <xacro:imu_sensor name="${name}_imu" parent="${name}_link" update_rate="100.0">
+    <xacro:imu_sensor name="${name}_imu" parent="${name}_link" update_rate="50.0">
       <origin xyz="0.200 0 0.200" rpy="0 ${0 * deg_to_rad} ${0 * deg_to_rad}"/>
     </xacro:imu_sensor>
@@ -81,4 +82,26 @@
     <xacro:caster side="back_left" radius="${caster_radius}" width="${caster_width}" position_x="-0.213" position_y="0.141" position_z="0.0971" offset_x="-0.030" offset_y="0" offset_z="-0.0596" parent="${name}"/>
     <xacro:caster side="back_right" radius="${caster_radius}" width="${caster_width}" position_x="-0.213" position_y="-0.141" position_z="0.0971" offset_x="-0.030" offset_y="0" offset_z="-0.0596" parent="${name}"/>
+    <!-- Sonar sensors -->
+    <xacro:sonar_sensor name="${name}_sonar_1" parent="${name}" ros_topic="sonar_1" update_rate="20" maxRange="4.0" minRange="0.01" fov="${35 * deg_to_rad}" radiation="ultrasound">
+      <origin xyz="0.2688 0.17956 0.06155" rpy="0 0 ${30 * deg_to_rad}"/>
+    </xacro:sonar_sensor>
+    <xacro:sonar_sensor name="${name}_sonar_2" parent="${name}" ros_topic="sonar_2" update_rate="20" maxRange="4.0" minRange="0.01" fov="${35 * deg_to_rad}" radiation="ultrasound">
+      <origin xyz="0.28947 0.09241 0.06155" rpy="0 0 ${12 * deg_to_rad}"/>
+    </xacro:sonar_sensor>
+    <xacro:sonar_sensor name="${name}_sonar_3" parent="${name}" ros_topic="sonar_3" update_rate="20" maxRange="4.0" minRange="0.01" fov="${35 * deg_to_rad}" radiation="ultrasound">
+      <origin xyz="0.29671 0.0 0.06155" rpy="0 0 ${0 * deg_to_rad}"/>
+    </xacro:sonar_sensor>
+    <xacro:sonar_sensor name="${name}_sonar_4" parent="${name}" ros_topic="sonar_4" update_rate="20" maxRange="4.0" minRange="0.01" fov="${35 * deg_to_rad}" radiation="ultrasound">
+      <origin xyz="0.28947 -0.09241 0.06155" rpy="0 0 ${-12 * deg_to_rad}"/>
+    </xacro:sonar_sensor>
+    <xacro:sonar_sensor name="${name}_sonar_5" parent="${name}" ros_topic="sonar_5" update_rate="20" maxRange="4.0" minRange="0.01" fov="${35 * deg_to_rad}" radiation="ultrasound">
+      <origin xyz="0.2688 -0.17956 0.06155" rpy="0 0 ${-30 * deg_to_rad}"/>
+    </xacro:sonar_sensor>
+    <xacro:sonar_sensor name="${name}_sonar_6" parent="${name}" ros_topic="sonar_6" update_rate="20" maxRange="4.0" minRange="0.01" fov="${35 * deg_to_rad}" radiation="ultrasound">
+      <origin xyz="-0.25648 -0.10103 0.28155" rpy="0 0 ${180 * deg_to_rad}"/>
+    </xacro:sonar_sensor>
+    <xacro:sonar_sensor name="${name}_sonar_7" parent="${name}" ros_topic="sonar_7" update_rate="20" maxRange="4.0" minRange="0.01" fov="${35 * deg_to_rad}" radiation="ultrasound">
+      <origin xyz="-0.25648 0.10103 0.28155" rpy="0 0 ${180 * deg_to_rad}"/>
+    </xacro:sonar_sensor>
   </xacro:macro>
 </robot>

File: mrp2_description/urdf/wheels/wheel.left.urdf.xacro (robot description, xacro)
@@ -36,5 +36,5 @@
       <parent link="${parent}_link"/>
       <child link="wheel_${side}_link"/>
-      <origin xyz="0 0.2395 ${radius}" rpy="0 0 0"/>
+      <origin xyz="0 ${separation / 2} ${radius}" rpy="0 0 0"/>
       <axis xyz="0 1 0"/>
       <limit effort="${torque*2}" velocity="${velocity / radius}"/>

File: mrp2_description/urdf/wheels/wheel.right.urdf.xacro (robot description, xacro)
@@ -36,5 +36,5 @@
       <parent link="${parent}_link"/>
       <child link="wheel_${side}_link"/>
-      <origin xyz="0 -0.2395 ${radius}" rpy="0 0 0"/>
+      <origin xyz="0 -${separation / 2} ${radius}" rpy="0 0 0"/>
       <axis xyz="0 1 0"/>
       <limit effort="${torque*2}" velocity="${velocity / radius}"/>

Commit message: Imported upstream version '0.2.3' of 'upstream'

File: mrp2_description/urdf/base/base.urdf.xacro (robot description, xacro)
@@ -11,5 +11,5 @@
   <property name="wheel_radius"     value="0.100"/>
   <property name="wheel_width"      value="0.050"/>
-  <property name="wheel_separation" value="0.478"/>
+  <property name="wheel_separation" value="0.4715"/>
   <property name="wheel_torque"     value="5.0"/>
   <property name="wheel_velocity"   value="2.0"/>
@@ -17,6 +17,6 @@
   <property name="caster_radius"       value="0.0375"/>
   <property name="caster_width"        value="0.020"/>
-  <property name="caster_separation_x" value="0.426"/>
-  <property name="caster_separation_y" value="0.282"/>
+  <property name="caster_separation_x" value="0.384"/>
+  <property name="caster_separation_y" value="0.288"/>
   <property name="caster_offset_x"     value="-0.002"/>
   <property name="caster_offset_y"     value="0.0"/>
@@ -25,5 +25,5 @@
   <property name="base_laser_x" value="0.239"/>
   <property name="base_laser_y" value="0.0"/>
-  <property name="base_laser_z" value="0.2581"/>
+  <property name="base_laser_z" value="0.2660"/>
   <xacro:macro name="base" params="name">
     <!-- Base -->
@@ -72,5 +72,5 @@
     <!-- IMU -->
     <xacro:imu_sensor name="${name}_imu" parent="${name}_link" update_rate="50.0">
-      <origin xyz="0.200 0 0.200" rpy="0 ${0 * deg_to_rad} ${0 * deg_to_rad}"/>
+      <origin xyz="0.1604 0 0.2440" rpy="0 ${0 * deg_to_rad} ${0 * deg_to_rad}"/>
     </xacro:imu_sensor>
     <!-- Wheels -->
@@ -78,8 +78,8 @@
     <xacro:wheel_left side="left"  reflect="1.0" radius="${wheel_radius}" width="${wheel_width}" torque="${wheel_torque}" velocity="${wheel_velocity}" separation="${wheel_separation}" parent="${name}"/>
     <!-- Casters wheels -->
-    <xacro:caster side="front_left" radius="${caster_radius}" width="${caster_width}" position_x="0.213" position_y="0.141" position_z="0.0971" offset_x="-0.030" offset_y="0" offset_z="-0.0596" parent="${name}"/>
-    <xacro:caster side="front_right" radius="${caster_radius}" width="${caster_width}" position_x="0.213" position_y="-0.141" position_z="0.0971" offset_x="-0.030" offset_y="0" offset_z="-0.0596" parent="${name}"/>
-    <xacro:caster side="back_left" radius="${caster_radius}" width="${caster_width}" position_x="-0.213" position_y="0.141" position_z="0.0971" offset_x="-0.030" offset_y="0" offset_z="-0.0596" parent="${name}"/>
-    <xacro:caster side="back_right" radius="${caster_radius}" width="${caster_width}" position_x="-0.213" position_y="-0.141" position_z="0.0971" offset_x="-0.030" offset_y="0" offset_z="-0.0596" parent="${name}"/>
+    <xacro:caster side="front_left" radius="${caster_radius}" width="${caster_width}" position_x="0.192" position_y="0.144" position_z="0.0971" offset_x="-0.030" offset_y="0" offset_z="-0.0596" parent="${name}"/>
+    <xacro:caster side="front_right" radius="${caster_radius}" width="${caster_width}" position_x="0.192" position_y="-0.144" position_z="0.0971" offset_x="-0.030" offset_y="0" offset_z="-0.0596" parent="${name}"/>
+    <xacro:caster side="back_left" radius="${caster_radius}" width="${caster_width}" position_x="-0.192" position_y="0.144" position_z="0.0971" offset_x="-0.030" offset_y="0" offset_z="-0.0596" parent="${name}"/>
+    <xacro:caster side="back_right" radius="${caster_radius}" width="${caster_width}" position_x="-0.192" position_y="-0.144" position_z="0.0971" offset_x="-0.030" offset_y="0" offset_z="-0.0596" parent="${name}"/>
     <!-- Sonar sensors -->
     <xacro:sonar_sensor name="${name}_sonar_1" parent="${name}" ros_topic="sonar_1" update_rate="20" maxRange="4.0" minRange="0.01" fov="${35 * deg_to_rad}" radiation="ultrasound">
