Commit message: Imported upstream version '1.0.1' of 'upstream'

File: mrp2_description/gazebo/gazebo.urdf.xacro (robot description, xacro)
@@ -1,19 +1,33 @@
 <?xml version="1.0"?>
-<robot xmlns:sensor="http://playerstage.sourceforge.net/gazebo/xmlschema/#sensor"
+<robot xmlns:xacro="http://www.ros.org/wiki/xacro"
+       xmlns:sensor="http://playerstage.sourceforge.net/gazebo/xmlschema/#sensor"
        xmlns:controller="http://playerstage.sourceforge.net/gazebo/xmlschema/#controller"
        xmlns:interface="http://playerstage.sourceforge.net/gazebo/xmlschema/#interface">
   <gazebo>
-    <plugin filename="libgazebo_ros_control.so" name="ros_control">
-      <ns></ns>
-      <robotSimType>mrp2_hardware_gazebo/Mrp2HardwareGazebo</robotSimType>
-      <controlPeriod>0.001</controlPeriod>
-    </plugin>
     <plugin filename="libgazebo_ros_p3d.so" name="gazebo_ros_p3d">
       <bodyName>base_footprint</bodyName>
       <topicName>ground_truth_odom</topicName>
       <alwaysOn>true</alwaysOn>
-      <updateRate>100.0</updateRate>
+      <updateRate>20</updateRate>
+    </plugin>
+    <plugin filename="libgazebo_ros_diff_drive.so" name="differential_drive_controller">
+      <updateRate>20</updateRate>
+      <leftJoint>wheel_left_joint</leftJoint>
+      <rightJoint>wheel_right_joint</rightJoint>
+      <wheelSeparation>0.5380</wheelSeparation>
+      <wheelDiameter>0.2410</wheelDiameter>
+      <wheelAcceleration>1.0</wheelAcceleration>
+      <wheelTorque>20</wheelTorque>
+      <commandTopic>cmd_vel</commandTopic>
+      <odometryTopic>odom</odometryTopic>
+      <odometryFrame>odom</odometryFrame>
+      <robotBaseFrame>base_footprint</robotBaseFrame>
+      <odometrySource>encoder</odometrySource>
+      <publishWheelTF>false</publishWheelTF>
+      <publishOdom>true</publishOdom>
+      <publishWheelJointState>true</publishWheelJointState>
+      <legacyMode>false</legacyMode>
     </plugin>
   </gazebo>
-  <property name="M_PI" value="3.14159" />
+  <xacro:property name="M_PI" value="3.14159" />
 </robot>

File: mrp2_description/urdf/base/base.urdf.xacro (robot description, xacro)
@@ -2,6 +2,5 @@
 <robot xmlns:xacro="http://ros.org/wiki/xacro">
   <xacro:include filename="$(find mrp2_description)/urdf/deg_to_rad.xacro"/>
-  <xacro:include filename="$(find mrp2_description)/urdf/wheels/wheel.right.urdf.xacro"/>
-  <xacro:include filename="$(find mrp2_description)/urdf/wheels/wheel.left.urdf.xacro"/>
+  <xacro:include filename="$(find mrp2_description)/urdf/wheels/wheel.urdf.xacro"/>
   <xacro:include filename="$(find mrp2_description)/urdf/wheels/75mm.caster.urdf.xacro"/>
   <xacro:include filename="$(find mrp2_description)/urdf/sensors/hokuyo_utm_30lx_laser.urdf.xacro"/>
@@ -9,21 +8,21 @@
   <xacro:include filename="$(find mrp2_description)/urdf/sensors/sonar.urdf.xacro"/>
   <!-- Wheel characteristics -->
-  <property name="wheel_radius"     value="0.100"/>
-  <property name="wheel_width"      value="0.050"/>
-  <property name="wheel_separation" value="0.4715"/>
-  <property name="wheel_torque"     value="5.0"/>
-  <property name="wheel_velocity"   value="2.0"/>
+  <xacro:property name="wheel_radius"     value="0.100"/>
+  <xacro:property name="wheel_width"      value="0.050"/>
+  <xacro:property name="wheel_separation" value="0.4715"/>
+  <xacro:property name="wheel_torque"     value="5.0"/>
+  <xacro:property name="wheel_velocity"   value="2.0"/>
   <!-- Caster wheel characteristics -->
-  <property name="caster_radius"       value="0.0375"/>
-  <property name="caster_width"        value="0.020"/>
-  <property name="caster_separation_x" value="0.384"/>
-  <property name="caster_separation_y" value="0.288"/>
-  <property name="caster_offset_x"     value="-0.002"/>
-  <property name="caster_offset_y"     value="0.0"/>
-  <property name="caster_offset_z"     value="0.075"/>
+  <xacro:property name="caster_radius"       value="0.0375"/>
+  <xacro:property name="caster_width"        value="0.020"/>
+  <xacro:property name="caster_separation_x" value="0.384"/>
+  <xacro:property name="caster_separation_y" value="0.288"/>
+  <xacro:property name="caster_offset_x"     value="-0.002"/>
+  <xacro:property name="caster_offset_y"     value="0.0"/>
+  <xacro:property name="caster_offset_z"     value="0.075"/>
   <!-- Laser characteristics -->
-  <property name="base_laser_x" value="0.239"/>
-  <property name="base_laser_y" value="0.0"/>
-  <property name="base_laser_z" value="0.2660"/>
+  <xacro:property name="base_laser_x" value="0.239"/>
+  <xacro:property name="base_laser_y" value="0.0"/>
+  <xacro:property name="base_laser_z" value="0.2660"/>
   <xacro:macro name="base" params="name">
     <!-- Base -->
@@ -67,14 +66,26 @@
       <parent link="${name}_footprint"/>
     </joint>
-    <xacro:hokuyo_utm_30lx_laser name="${name}_laser" parent="${name}" ros_topic="scan" update_rate="10" min_angle="${-135 * deg_to_rad}" max_angle="${135 * deg_to_rad}" >
+    <xacro:hokuyo_utm_30lx_laser name="${name}_laser" parent="${name}" ros_topic="scan" update_rate="20" min_angle="${-135 * deg_to_rad}" max_angle="${135 * deg_to_rad}" >
       <origin xyz="${base_laser_x} ${base_laser_y} ${base_laser_z}" rpy="0 0 0" />
     </xacro:hokuyo_utm_30lx_laser>
-    <!-- IMU -->
-    <xacro:imu_sensor name="${name}_imu" parent="${name}_link" update_rate="50.0">
-      <origin xyz="0.1604 0 0.2440" rpy="0 ${0 * deg_to_rad} ${0 * deg_to_rad}"/>
-    </xacro:imu_sensor>
     <!-- Wheels -->
-    <xacro:wheel_right side="right" reflect="-1.0" radius="${wheel_radius}" width="${wheel_width}" torque="${wheel_torque}" velocity="${wheel_velocity}" separation="${wheel_separation}" parent="${name}"/>
-    <xacro:wheel_left side="left"  reflect="1.0" radius="${wheel_radius}" width="${wheel_width}" torque="${wheel_torque}" velocity="${wheel_velocity}" separation="${wheel_separation}" parent="${name}"/>
+    <xacro:wheel
+      side="right"
+      reflect="-1.0"
+      radius="${wheel_radius}"
+      width="${wheel_width}"
+      torque="${wheel_torque}"
+      velocity="${wheel_velocity}"
+      separation="-${wheel_separation}"
+      parent="${name}_link"/>
+    <xacro:wheel
+      side="left"
+      reflect="1.0"
+      radius="${wheel_radius}"
+      width="${wheel_width}"
+      torque="${wheel_torque}"
+      velocity="${wheel_velocity}"
+      separation="${wheel_separation}"
+      parent="${name}_link"/>
     <!-- Casters wheels -->
     <xacro:caster side="front_left" radius="${caster_radius}" width="${caster_width}" position_x="0.192" position_y="0.144" position_z="0.0971" offset_x="-0.030" offset_y="0" offset_z="-0.0596" parent="${name}"/>
@@ -82,4 +93,8 @@
     <xacro:caster side="back_left" radius="${caster_radius}" width="${caster_width}" position_x="-0.192" position_y="0.144" position_z="0.0971" offset_x="-0.030" offset_y="0" offset_z="-0.0596" parent="${name}"/>
     <xacro:caster side="back_right" radius="${caster_radius}" width="${caster_width}" position_x="-0.192" position_y="-0.144" position_z="0.0971" offset_x="-0.030" offset_y="0" offset_z="-0.0596" parent="${name}"/>
+    <!-- IMU -->
+    <xacro:imu_sensor name="${name}_imu" parent="${name}_link" update_rate="20.0">
+      <origin xyz="0.1604 0 0.2440" rpy="0 ${0 * deg_to_rad} ${0 * deg_to_rad}"/>
+    </xacro:imu_sensor>
     <!-- Sonar sensors -->
     <xacro:sonar_sensor name="${name}_sonar_1" parent="${name}" ros_topic="sonar_1" update_rate="20" maxRange="4.0" minRange="0.01" fov="${35 * deg_to_rad}" radiation="ultrasound">

File: mrp2_description/urdf/sensors/hokuyo_urg_04lx_ug01_laser.urdf.xacro (robot description, xacro)
@@ -21,5 +21,5 @@
     <joint name="${name}_joint" type="fixed">
       <axis xyz="0 1 0"/>
-      <insert_block name="origin"/>
+      <xacro:insert_block name="origin"/>
       <parent link="${parent}_link"/>
       <child  link="${name}_link"/>

File: mrp2_description/urdf/sensors/hokuyo_utm_30lx_laser.urdf.xacro (robot description, xacro)
@@ -21,5 +21,5 @@
     <joint name="${name}_joint" type="fixed">
       <axis xyz="0 1 0"/>
-      <insert_block name="origin"/>
+      <xacro:insert_block name="origin"/>
       <parent link="${parent}_link"/>
       <child  link="${name}_link"/>

File: mrp2_description/urdf/sensors/imu.urdf.xacro (robot description, xacro)
@@ -12,11 +12,21 @@
       <parent link="${parent}"/>
       <child link="${name}_link"/>
-      <insert_block name="origin"/>
+      <xacro:insert_block name="origin"/>
     </joint>
     <gazebo reference="${name}_link">
       <sensor name="${name}_sensor" type="imu">
         <always_on>1</always_on>
-        <update_rate>100.0</update_rate>
-        <imu>
+        <update_rate>20.0</update_rate>
+        <plugin filename="libgazebo_ros_imu_sensor.so" name="imu_plugin">
+          <topicName>imu</topicName>
+          <bodyName>base_imu_link</bodyName>
+          <updateRateHZ>20.0</updateRateHZ>
+          <gaussianNoise>0.0</gaussianNoise>
+          <xyzOffset>0 0 0</xyzOffset>
+          <rpyOffset>0 0 0</rpyOffset>
+          <frameName>base_imu_link</frameName>
+          <initialOrientationAsReference>false</initialOrientationAsReference>
+        </plugin>
+        <!--imu>
           <noise>
             <type>gaussian</type>
@@ -34,5 +44,5 @@
             </accel>
           </noise>
-        </imu>
+        </imu-->
       </sensor>
     </gazebo>

File: mrp2_description/urdf/sensors/sonar.urdf.xacro (robot description, xacro)
@@ -20,5 +20,5 @@
     </link>
     <joint name="${name}_joint" type="fixed">
-      <insert_block name="origin"/>
+      <xacro:insert_block name="origin"/>
       <axis xyz="0 0 1"/>
       <parent link="${parent}_link"/>
